File: kicad/kicad.kicad_pcb (KiCad board)
At the start: 2 copper layers, 9 parts, among them M1 DC Motor (w/ Encoders), M2 DC Motor (w/ Encoders), M3 DC Motor (w/ Encoders)

Commit message: pcb mostly finished
Parts:
- removed DRIVER0: TB6612FNG, Connector_PinHeader_2.54mm:PinHeader_1x08_P2.54mm_Vertical
- added DRIVER2: TB6612FNG, Breakout_Board:Motor_Driver_Breakout, F.Cu at (152.0, 59.4)
- DRIVER1: footprint Connector_PinHeader_2.54mm:PinHeader_1x08_P2.54mm_Vertical -> Breakout_Board:Motor_Driver_Breakout
- M1, M2, M3: footprint Connector_PinHeader_1.00mm:PinHeader_1x03_P1.00mm_Vertical -> Breakout_Board:Untitled_1
- SENSOR0, SENSOR1, SENSOR2: footprint Connector_PinSocket_2.54mm:PinSocket_1x03_P2.54mm_Vertical -> Breakout_Board:Untitled_1
- moved SENSOR0 98.4 mm to (113.5, 30.4), turned to 0 degrees
- moved M2 92.7 mm to (170.9, 29.9)
- moved SENSOR1 83.1 mm to (113.5, 43.0), turned to 0 degrees
- moved SENSOR2 72.8 mm to (113.0, 56.6), turned to 0 degrees
- moved M1 67.5 mm to (179.0, 57.6), turned to 180 degrees
- moved DRIVER1 58.2 mm to (152.0, 84.3), turned to 180 degrees
- moved M3 51.8 mm to (178.5, 75.6), turned to 180 degrees
- moved RPIPICOW1 35.3 mm to (142.5, 82.0), turned to 180 degrees
Connections:
- DRIVER1 pad 1: Net-(M3-+) -> Net-(DRIVER1A-PWMA)
- DRIVER1 pad 2: Net-(M3-+) -> Net-(DRIVER1A-AIN2)
- DRIVER1 pad 3: unconnected-(DRIVER1A-PGND1-Pad3)_1 -> Net-(DRIVER1A-AIN1)
- DRIVER1 pad 4: unconnected-(DRIVER1A-PGND1-Pad3) -> Net-(DRIVER1A-STBY)
- DRIVER1 pad 5: Net-(M3--) -> unconnected-(DRIVER1A-BIN1-Pad5)
- M1 pad 3: (no net) -> Net-(M1-EN)
- M2 pad 3: (no net) -> Net-(M2-EN)
- M3 pad 3: (no net) -> Net-(M3-EN)
Routing:
- net GNDREF: track 0.00 -> 273.1 mm
- net +3V0: track 0.00 -> 209.7 mm
- net +3V3: track 0.00 -> 98.4 mm
- net Net-(M1-EN): track 0.00 -> 71.1 mm
- net Net-(M2-EN): track 0.00 -> 67.3 mm
- net Net-(DRIVER1A-PWMA): track 0.00 -> 51.2 mm
- net Net-(M3-EN): track 0.00 -> 40.9 mm
- net +12V: track 0.00 -> 39.1 mm
- net Net-(DRIVER1A-STBY): track 0.00 -> 37.5 mm
- net Net-(DRIVER2A-STBY): track 0.00 -> 35.7 mm
- net Net-(DRIVER1A-AIN2): track 0.00 -> 29.0 mm
- net Net-(DRIVER2A-PWMB): track 0.00 -> 28.1 mm
- net Net-(DRIVER2A-PWMA): track 0.00 -> 26.3 mm
- net Net-(DRIVER1A-AIN1): track 0.00 -> 26.0 mm
- net Net-(RPIPICOW1-GPIO26_ADC0): track 0.00 -> 22.7 mm
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
Commit message: pcb edits and flip
Parts:
- moved SENSOR0 95.3 mm to (174.5, 103.6), turned to 180 degrees
- moved M2 91.6 mm to (117.0, 104.0), turned to 180 degrees
- moved SENSOR1 77.8 mm to (174.6, 91.0), turned to 180 degrees
- moved M1 72.5 mm to (109.0, 76.4), turned to 0 degrees
- moved M3 71.1 mm to (109.5, 58.4), turned to 0 degrees
- moved SENSOR2 65.4 mm to (175.0, 77.4), turned to 180 degrees
- moved DRIVER1 38.1 mm to (136.0, 49.7), turned to 0 degrees
- moved RPIPICOW1 30.2 mm to (145.5, 52.0), turned to 0 degrees
- moved DRIVER2 22.1 mm to (136.0, 74.6), turned to 0 degrees
Routing:
- net +3V3: track 98.4 -> 102.5 mm
- net GNDREF: track 273.1 -> 275.5 mm
Other:
- board text added: "DC Motor (w/ Encoders)"
- board text added: "DRIVER1"
- board text added: "DRIVER2"

Commit message: upload updated kiCAD files
Parts:
- moved M1 3.09 mm to (111.8, 75.1)
- moved M2 2.88 mm to (119.8, 104.9)
- moved M3 2.33 mm to (111.8, 58.8)
Routing:
- net +3V0: track 209.3 -> 153.4 mm
- net GNDREF: track 275.5 -> 289.9 mm
- net +12V: track 39.1 -> 27.1 mm
- net Net-(M2-EN): track 67.8 -> 57.4 mm
- net Net-(M1-EN): track 71.5 -> 63.6 mm
- net Net-(DRIVER2A-AIN1): track 16.0 -> 8.74 mm
- net +3V3: track 102.5 -> 95.6 mm
- net Net-(M1--): track 15.4 -> 10.8 mm
- net Net-(M1-+): track 15.4 -> 11.5 mm
- net Net-(M3-EN): track 40.9 -> 37.8 mm
- net Net-(M2-+): track 10.5 -> 8.07 mm
- net Net-(M2--): track 10.5 -> 8.07 mm
- net Net-(M3--): track 10.3 -> 8.16 mm
- net Net-(M3-+): track 10.3 -> 8.16 mm
- net Net-(DRIVER1A-AIN1): track 26.0 -> 24.9 mm
Other:
- board outline added: 99.5 x 60.4 mm
- board text added: "+"
- board text added: "-"
- board text added: "M1"
- board text added: "M2"
- board text added: "M3"
- board text added: "SIG"
- board text removed: "DC Motor (w/ Encoders)"
